Commit message: add pipe to env

File: install/simple_car_sim/share/simple_car_sim/urdf/robot.urdf.xacro (robot description, xacro)
@@ -1,95 +1 @@
-<?xml version="1.0"?>
-<robot xmlns:xacro="http://www.ros.org/wiki/xacro" name="simple_car">
-  <!-- Inertial Macros -->
-  <xacro:macro name="box_inertia" params="m x y z">
-    <inertial>
-      <mass value="${m}"/>
-      <inertia ixx="${m*(y*y+z*z)/12}" ixy="0" ixz="0"
-               iyy="${m*(x*x+z*z)/12}" iyz="0"
-               izz="${m*(x*x+y*y)/12}"/>
-    </inertial>
-  </xacro:macro>
-  <xacro:macro name="cylinder_inertia" params="m r h">
-    <inertial>
-      <mass value="${m}"/>
-      <inertia ixx="${m*(3*r*r+h*h)/12}" ixy="0" ixz="0"
-               iyy="${m*(3*r*r+h*h)/12}" iyz="0"
-               izz="${m*r*r/2}"/>
-    </inertial>
-  </xacro:macro>
-  <!-- Base Link -->
-  <link name="base_link">
-    <visual>
-      <geometry>
-        <box size="0.5 0.3 0.1"/>
-      </geometry>
-      <material name="blue">
-        <color rgba="0 0 1 1"/>
-      </material>
-    </visual>
-    <collision>
-      <geometry>
-        <box size="0.5 0.3 0.1"/>
-      </geometry>
-    </collision>
-    <xacro:box_inertia m="5.0" x="0.5" y="0.3" z="0.1"/>
-  </link>
-  <!-- Wheels -->
-  <xacro:macro name="wheel" params="name x y">
-    <link name="${name}_wheel">
-      <visual>
-        <geometry>
-          <cylinder radius="0.1" length="0.05"/>
-        </geometry>
-        <material name="black">
-          <color rgba="0 0 0 1"/>
-        </material>
-      </visual>
-      <collision>
-        <geometry>
-          <cylinder radius="0.1" length="0.05"/>
-        </geometry>
-        <surface>
-          <friction>
-            <ode>
-              <mu>0.5</mu>
-              <mu2>0.5</mu2>
-            </ode>
-          </friction>
-        </surface>
-      </collision>
-      <xacro:cylinder_inertia m="1.0" r="0.1" h="0.05"/>
-    </link>
-    <joint name="${name}_wheel_joint" type="continuous">
-      <parent link="base_link"/>
-      <child link="${name}_wheel"/>
-      <origin xyz="${x} ${y} -0.05" rpy="-1.5707 0 0"/>
-      <axis xyz="0 0 1"/>
-    </joint>
-  </xacro:macro>
-  <!-- Increased y offset to avoid collision with base_link (0.15 + 0.025 + gap) -->
-  <xacro:wheel name="front_left" x="0.15" y="0.2"/>
-  <xacro:wheel name="front_right" x="0.15" y="-0.2"/>
-  <xacro:wheel name="rear_left" x="-0.15" y="0.2"/>
-  <xacro:wheel name="rear_right" x="-0.15" y="-0.2"/>
-  <!-- Gazebo Plugin for Diff Drive (Skid Steer style) -->
-  <gazebo>
-    <plugin filename="ignition-gazebo-diff-drive-system" name="ignition::gazebo::systems::DiffDrive">
-      <left_joint>front_left_wheel_joint</left_joint>
-      <left_joint>rear_left_wheel_joint</left_joint>
-      <right_joint>front_right_wheel_joint</right_joint>
-      <right_joint>rear_right_wheel_joint</right_joint>
-      <wheel_separation>0.4</wheel_separation>
-      <wheel_radius>0.1</wheel_radius>
-      <odom_publish_frequency>20</odom_publish_frequency>
-      <topic>cmd_vel</topic>
-      <odom_topic>odom</odom_topic>
-      <tf_topic>tf</tf_topic>
-      <frame_id>odom</frame_id>
-      <child_frame_id>base_link</child_frame_id>
-    </plugin>
-    <!-- Joint State Publisher -->
-    <plugin filename="ignition-gazebo-joint-state-publisher-system" name="ignition::gazebo::systems::JointStatePublisher">
-    </plugin>
-  </gazebo>
-</robot>
+/home/yinyudream/Desktop/final_design/src/simple_car_sim/urdf/robot.urdf.xacro

Commit message: add whell seed control

File: install/simple_car_sim/share/simple_car_sim/urdf/robot.urdf.xacro (robot description, xacro)
@@ -1 +1,102 @@
-/home/yinyudream/Desktop/final_design/src/simple_car_sim/urdf/robot.urdf.xacro
+<?xml version="1.0"?>
+<robot xmlns:xacro="http://www.ros.org/wiki/xacro" name="simple_car">
+  <!-- Inertial Macros -->
+  <xacro:macro name="box_inertia" params="m x y z">
+    <inertial>
+      <mass value="${m}"/>
+      <inertia ixx="${m*(y*y+z*z)/12}" ixy="0" ixz="0"
+               iyy="${m*(x*x+z*z)/12}" iyz="0"
+               izz="${m*(x*x+y*y)/12}"/>
+    </inertial>
+  </xacro:macro>
+  <xacro:macro name="cylinder_inertia" params="m r h">
+    <inertial>
+      <mass value="${m}"/>
+      <inertia ixx="${m*(3*r*r+h*h)/12}" ixy="0" ixz="0"
+               iyy="${m*(3*r*r+h*h)/12}" iyz="0"
+               izz="${m*r*r/2}"/>
+    </inertial>
+  </xacro:macro>
+  <!-- Base Link -->
+  <link name="base_link">
+    <visual>
+      <geometry>
+        <box size="0.5 0.3 0.1"/>
+      </geometry>
+      <material name="blue">
+        <color rgba="0 0 1 1"/>
+      </material>
+    </visual>
+    <collision>
+      <geometry>
+        <box size="0.5 0.3 0.1"/>
+      </geometry>
+    </collision>
+    <xacro:box_inertia m="5.0" x="0.5" y="0.3" z="0.1"/>
+  </link>
+  <!-- Wheels -->
+  <xacro:macro name="wheel" params="name x y">
+    <link name="${name}_wheel">
+      <visual>
+        <geometry>
+          <cylinder radius="0.1" length="0.05"/>
+        </geometry>
+        <material name="black">
+          <color rgba="0 0 0 1"/>
+        </material>
+      </visual>
+      <collision>
+        <geometry>
+          <cylinder radius="0.1" length="0.05"/>
+        </geometry>
+        <surface>
+          <friction>
+            <ode>
+              <mu>100.0</mu>
+              <mu2>100.0</mu2>
+              <fdir1>1 0 0</fdir1>
+              <slip1>0.0</slip1>
+              <slip2>0.0</slip2>
+            </ode>
+          </friction>
+          <contact>
+            <ode>
+              <min_depth>0.005</min_depth>
+              <kp>1e8</kp>
+            </ode>
+          </contact>
+        </surface>
+      </collision>
+      <xacro:cylinder_inertia m="1.0" r="0.1" h="0.05"/>
+    </link>
+    <joint name="${name}_wheel_joint" type="continuous">
+      <parent link="base_link"/>
+      <child link="${name}_wheel"/>
+      <origin xyz="${x} ${y} -0.05" rpy="-1.5707 0 0"/>
+      <axis xyz="0 0 1"/>
+    </joint>
+  </xacro:macro>
+  <!-- Increased y offset to avoid collision with base_link (0.15 + 0.025 + gap) -->
+  <xacro:wheel name="front_left" x="0.15" y="0.2"/>
+  <xacro:wheel name="front_right" x="0.15" y="-0.2"/>
+  <xacro:wheel name="rear_left" x="-0.15" y="0.2"/>
+  <xacro:wheel name="rear_right" x="-0.15" y="-0.2"/>
+  <!-- Gazebo Plugins for Joint Control -->
+  <gazebo>
+    <plugin filename="ignition-gazebo-joint-controller-system" name="ignition::gazebo::systems::JointController">
+      <joint_name>front_left_wheel_joint</joint_name>
+    </plugin>
+    <plugin filename="ignition-gazebo-joint-controller-system" name="ignition::gazebo::systems::JointController">
+      <joint_name>rear_left_wheel_joint</joint_name>
+    </plugin>
+    <plugin filename="ignition-gazebo-joint-controller-system" name="ignition::gazebo::systems::JointController">
+      <joint_name>front_right_wheel_joint</joint_name>
+    </plugin>
+    <plugin filename="ignition-gazebo-joint-controller-system" name="ignition::gazebo::systems::JointController">
+      <joint_name>rear_right_wheel_joint</joint_name>
+    </plugin>
+    <!-- Joint State Publisher -->
+    <plugin filename="ignition-gazebo-joint-state-publisher-system" name="ignition::gazebo::systems::JointStatePublisher">
+    </plugin>
+  </gazebo>
+</robot>

File: src/simple_car_sim/urdf/robot.urdf.xacro (robot description, xacro)
@@ -53,8 +53,17 @@
           <friction>
             <ode>
-              <mu>0.5</mu>
-              <mu2>0.5</mu2>
+              <mu>100.0</mu>
+              <mu2>100.0</mu2>
+              <fdir1>1 0 0</fdir1>
+              <slip1>0.0</slip1>
+              <slip2>0.0</slip2>
             </ode>
           </friction>
+          <contact>
+            <ode>
+              <min_depth>0.005</min_depth>
+              <kp>1e8</kp>
+            </ode>
+          </contact>
         </surface>
       </collision>
@@ -73,19 +82,17 @@
   <xacro:wheel name="rear_left" x="-0.15" y="0.2"/>
   <xacro:wheel name="rear_right" x="-0.15" y="-0.2"/>
-  <!-- Gazebo Plugin for Diff Drive (Skid Steer style) -->
+  <!-- Gazebo Plugins for Joint Control -->
   <gazebo>
-    <plugin filename="ignition-gazebo-diff-drive-system" name="ignition::gazebo::systems::DiffDrive">
-      <left_joint>front_left_wheel_joint</left_joint>
-      <left_joint>rear_left_wheel_joint</left_joint>
-      <right_joint>front_right_wheel_joint</right_joint>
-      <right_joint>rear_right_wheel_joint</right_joint>
-      <wheel_separation>0.4</wheel_separation>
-      <wheel_radius>0.1</wheel_radius>
-      <odom_publish_frequency>20</odom_publish_frequency>
-      <topic>cmd_vel</topic>
-      <odom_topic>odom</odom_topic>
-      <tf_topic>tf</tf_topic>
-      <frame_id>odom</frame_id>
-      <child_frame_id>base_link</child_frame_id>
+    <plugin filename="ignition-gazebo-joint-controller-system" name="ignition::gazebo::systems::JointController">
+      <joint_name>front_left_wheel_joint</joint_name>
+    </plugin>
+    <plugin filename="ignition-gazebo-joint-controller-system" name="ignition::gazebo::systems::JointController">
+      <joint_name>rear_left_wheel_joint</joint_name>
+    </plugin>
+    <plugin filename="ignition-gazebo-joint-controller-system" name="ignition::gazebo::systems::JointController">
+      <joint_name>front_right_wheel_joint</joint_name>
+    </plugin>
+    <plugin filename="ignition-gazebo-joint-controller-system" name="ignition::gazebo::systems::JointController">
+      <joint_name>rear_right_wheel_joint</joint_name>
     </plugin>
     <!-- Joint State Publisher -->

Commit message: add sensors

File: install/simple_car_sim/share/simple_car_sim/urdf/robot.urdf.xacro (robot description, xacro)
@@ -82,6 +82,45 @@
   <xacro:wheel name="rear_left" x="-0.15" y="0.2"/>
   <xacro:wheel name="rear_right" x="-0.15" y="-0.2"/>
+  <!-- IMU Sensor -->
+  <link name="imu_link">
+    <visual>
+      <geometry>
+        <box size="0.05 0.05 0.05"/>
+      </geometry>
+      <material name="black">
+        <color rgba="0 0 0 1"/>
+      </material>
+    </visual>
+    <collision>
+      <geometry>
+        <box size="0.05 0.05 0.05"/>
+      </geometry>
+    </collision>
+    <xacro:box_inertia m="0.1" x="0.05" y="0.05" z="0.05"/>
+  </link>
+  <joint name="imu_joint" type="fixed">
+    <parent link="base_link"/>
+    <child link="imu_link"/>
+    <origin xyz="0 0 0.1" rpy="0 0 0"/>
+  </joint>
+  <gazebo reference="imu_link">
+    <sensor name="imu_sensor" type="imu">
+      <always_on>1</always_on>
+      <update_rate>100</update_rate>
+      <visualize>true</visualize>
+      <topic>imu</topic>
+    </sensor>
+  </gazebo>
   <!-- Gazebo Plugins for Joint Control -->
   <gazebo>
+    <!-- IMU Plugin -->
+    <plugin filename="ignition-gazebo-imu-system" name="ignition::gazebo::systems::Imu">
+    </plugin>
+    <!-- Odometry Publisher (Ground Truth) -->
+    <plugin filename="ignition-gazebo-odometry-publisher-system" name="ignition::gazebo::systems::OdometryPublisher">
+      <odom_frame>odom</odom_frame>
+      <robot_base_frame>base_link</robot_base_frame>
+      <dimensions>3</dimensions>
+    </plugin>
     <plugin filename="ignition-gazebo-joint-controller-system" name="ignition::gazebo::systems::JointController">
       <joint_name>front_left_wheel_joint</joint_name>
