Commit message: 1217 version

File: src/simple_car_sim/urdf/robot.urdf.xacro (robot description, xacro)
@@ -90,7 +90,21 @@
             <axis xyz="0 0 1"/> <!-- 沿局部Z轴伸缩 -->
             <limit lower="0.0" upper="0.8" effort="5000.0" velocity="0.5"/>
-        </joint>
-        <!-- 驱动轮 -->
-        <link name="drive_wheel_${location}_link">
+            <dynamics damping="5.0" friction="0.5"/>
+        </joint>
+        <!-- Bogie Link (连接两个轮子的支架) -->
+        <link name="drive_bogie_${location}_link">
+            <visual>
+                <geometry><box size="0.6 0.05 0.05"/></geometry>
+                <material name="grey"/>
+            </visual>
+            <xacro:box_inertial mass="0.5" x="0.6" y="0.05" z="0.05"/>
+        </link>
+        <joint name="drive_bogie_joint_${location}" type="fixed">
+            <parent link="drive_leg_${location}_link"/>
+            <child link="drive_bogie_${location}_link"/>
+            <origin xyz="0 0 0.1" rpy="0 0 0"/>
+        </joint>
+        <!-- Front Wheel -->
+        <link name="drive_wheel_${location}_front_link">
             <visual>
                 <geometry><cylinder radius="${wheel_radius}" length="${wheel_width}"/></geometry>
@@ -99,22 +113,51 @@
             </visual>
             <collision>
+                <geometry><sphere radius="${wheel_radius}"/></geometry>
+                <origin rpy="${pi/2} 0 0"/>
+            </collision>
+            <xacro:cylinder_inertial mass="${mass_wheel}" r="${wheel_radius}" h="${wheel_width}"/>
+        </link>
+        <gazebo reference="drive_wheel_${location}_front_link">
+            <mu1>4.0</mu1>
+            <mu2>4.0</mu2>
+            <kp>10000.0</kp>
+            <kd>5.0</kd>
+            <minDepth>0.001</minDepth>
+        </gazebo>
+        <joint name="drive_wheel_${location}_front_joint" type="continuous">
+            <parent link="drive_bogie_${location}_link"/>
+            <child link="drive_wheel_${location}_front_link"/>
+            <origin xyz="0.25 0 0" rpy="0 0 0"/>
+            <axis xyz="0 1 0"/>
+            <limit effort="1000.0" velocity="20.0"/>
+            <dynamics damping="0.5" friction="0.2"/>
+        </joint>
+        <!-- Rear Wheel -->
+        <link name="drive_wheel_${location}_rear_link">
+            <visual>
                 <geometry><cylinder radius="${wheel_radius}" length="${wheel_width}"/></geometry>
                 <origin rpy="${pi/2} 0 0"/>
+                <material name="black"/>
+            </visual>
+            <collision>
+                <geometry><sphere radius="${wheel_radius}"/></geometry>
+                <origin rpy="${pi/2} 0 0"/>
             </collision>
             <xacro:cylinder_inertial mass="${mass_wheel}" r="${wheel_radius}" h="${wheel_width}"/>
         </link>
-        <gazebo reference="drive_wheel_${location}_link">
-            <mu1>100.0</mu1>
-            <mu2>100.0</mu2>
-            <kp>1000000.0</kp>
-            <kd>1.0</kd>
+        <gazebo reference="drive_wheel_${location}_rear_link">
+            <mu1>4.0</mu1>
+            <mu2>4.0</mu2>
+            <kp>10000.0</kp>
+            <kd>5.0</kd>
             <minDepth>0.001</minDepth>
         </gazebo>
-        <!-- 驱动关节 -->
-        <joint name="drive_wheel_${location}_joint" type="continuous">
-            <parent link="drive_leg_${location}_link"/>
-            <child link="drive_wheel_${location}_link"/>
-            <origin xyz="0 0 0.1" rpy="0 0 0"/> <!-- 安装在腿的末端 -->
+        <joint name="drive_wheel_${location}_rear_joint" type="continuous">
+            <parent link="drive_bogie_${location}_link"/>
+            <child link="drive_wheel_${location}_rear_link"/>
+            <origin xyz="-0.25 0 0" rpy="0 0 0"/>
             <axis xyz="0 1 0"/>
+            <limit effort="1000.0" velocity="20.0"/>
+            <dynamics damping="0.5" friction="0.2"/>
         </joint>
     </xacro:macro>
@@ -145,9 +188,11 @@
         <origin xyz="-${body_len/2 + 0.08} 0 0" rpy="0 0 0"/>
         <axis xyz="0 1 0"/>
-        <limit lower="-0.8" upper="0.8" effort="100.0" velocity="0.5"/>
+        <limit lower="-1.57" upper="1.57" effort="100.0" velocity="0.5"/>
+        <dynamics damping="3.0" friction="0.2"/>
     </joint>
     <!-- 功能节的主体基座 -->
     <link name="func_base_link">
         <visual>
+            <origin xyz="-${body_len/2} 0 0" rpy="0 0 0"/> <!-- Offset geometry to start after joint -->
             <geometry>
                 <box size="${body_len} ${body_width} ${body_height}"/>
@@ -156,4 +201,5 @@
         </visual>
         <collision>
+            <origin xyz="-${body_len/2} 0 0" rpy="0 0 0"/>
             <geometry>
                 <box size="${body_len} ${body_width} ${body_height}"/>
@@ -168,5 +214,6 @@
         <origin xyz="-0.12 0 0" rpy="0 0 0"/>
         <axis xyz="0 0 1"/>
-        <limit lower="-0.8" upper="0.8" effort="100.0" velocity="0.5"/>
+        <limit lower="-1.57" upper="1.57" effort="100.0" velocity="0.5"/>
+        <dynamics damping="3.0" friction="0.2"/>
     </joint>
     <!-- ========================================================== -->
@@ -202,31 +249,63 @@
             <axis xyz="0 0 1"/>
             <limit lower="0.0" upper="0.8" effort="5000.0" velocity="0.5"/>
-        </joint>
-        <!-- 被动轮 (Passive Wheel) -->
-        <link name="passive_wheel_${suffix}_link">
-            <visual>
-                <geometry>
-                    <sphere radius="0.04"/> <!-- 简化为球轮 -->
-                </geometry>
+            <dynamics damping="5.0" friction="0.5"/>
+        </joint>
+        <!-- Bogie Link (连接两个轮子的支架) -->
+        <link name="passive_bogie_${suffix}_link">
+            <visual>
+                <geometry><box size="0.4 0.05 0.05"/></geometry>
+                <material name="grey"/>
+            </visual>
+            <xacro:box_inertial mass="0.5" x="0.4" y="0.05" z="0.05"/>
+        </link>
+        <joint name="passive_bogie_joint_${suffix}" type="fixed">
+            <parent link="leg_${suffix}_link"/>
+            <child link="passive_bogie_${suffix}_link"/>
+            <origin xyz="0 0 ${leg_length}" rpy="0 0 0"/>
+        </joint>
+        <!-- Front Passive Wheel -->
+        <link name="passive_wheel_${suffix}_front_link">
+            <visual>
+                <geometry><sphere radius="0.04"/></geometry>
                 <material name="black"/>
             </visual>
              <collision>
-                <geometry>
-                    <sphere radius="0.04"/>
-                </geometry>
+                <geometry><sphere radius="0.04"/></geometry>
             </collision>
             <xacro:box_inertial mass="0.1" x="0.08" y="0.08" z="0.08"/>
         </link>
-        <gazebo reference="passive_wheel_${suffix}_link">
-            <mu1>0.1</mu1> <!-- 被动轮摩擦力小一点，方便滑动? 不，它是支撑轮，应该也要有摩擦力防止打滑，但如果是万向轮... 这里简化为球轮 -->
-            <mu2>0.1</mu2>
+        <gazebo reference="passive_wheel_${suffix}_front_link">
+            <mu1>0.001</mu1>
+            <mu2>0.001</mu2>
             <kp>1000000.0</kp>
             <kd>1.0</kd>
         </gazebo>
-        <!-- 轮子关节 (Continuous) -->
-        <joint name="passive_wheel_joint_${suffix}" type="continuous">
-            <parent link="leg_${suffix}_link"/>
-            <child link="passive_wheel_${suffix}_link"/>
-            <origin xyz="0 0 ${leg_length}" rpy="0 0 0"/>
+        <joint name="passive_wheel_joint_${suffix}_front" type="continuous">
+            <parent link="passive_bogie_${suffix}_link"/>
+            <child link="passive_wheel_${suffix}_front_link"/>
+            <origin xyz="0.15 0 0" rpy="0 0 0"/>
+            <axis xyz="0 1 0"/>
+        </joint>
+        <!-- Rear Passive Wheel -->
+        <link name="passive_wheel_${suffix}_rear_link">
+            <visual>
+                <geometry><sphere radius="0.04"/></geometry>
+                <material name="black"/>
+            </visual>
+             <collision>
+                <geometry><sphere radius="0.04"/></geometry>
+            </collision>
+            <xacro:box_inertial mass="0.1" x="0.08" y="0.08" z="0.08"/>
+        </link>
+        <gazebo reference="passive_wheel_${suffix}_rear_link">
+            <mu1>0.001</mu1>
+            <mu2>0.001</mu2>
+            <kp>1000000.0</kp>
+            <kd>1.0</kd>
+        </gazebo>
+        <joint name="passive_wheel_joint_${suffix}_rear" type="continuous">
+            <parent link="passive_bogie_${suffix}_link"/>
+            <child link="passive_wheel_${suffix}_rear_link"/>
+            <origin xyz="-0.15 0 0" rpy="0 0 0"/>
             <axis xyz="0 1 0"/>
         </joint>
@@ -247,11 +326,15 @@
         <!-- Drive Wheels Controller -->
         <plugin filename="libignition-gazebo-joint-controller-system.so" name="ignition::gazebo::systems::JointController">
-            <joint_name>drive_wheel_top_joint</joint_name>
-            <joint_name>drive_wheel_bottom_joint</joint_name>
-            <joint_name>drive_wheel_left_joint</joint_name>
-            <joint_name>drive_wheel_right_joint</joint_name>
-            <p_gain>1.0</p_gain>
-            <i_gain>0.1</i_gain>
-            <d_gain>0.01</d_gain>
+            <joint_name>drive_wheel_top_front_joint</joint_name>
+            <joint_name>drive_wheel_top_rear_joint</joint_name>
+            <joint_name>drive_wheel_bottom_front_joint</joint_name>
+            <joint_name>drive_wheel_bottom_rear_joint</joint_name>
+            <joint_name>drive_wheel_left_front_joint</joint_name>
+            <joint_name>drive_wheel_left_rear_joint</joint_name>
+            <joint_name>drive_wheel_right_front_joint</joint_name>
+            <joint_name>drive_wheel_right_rear_joint</joint_name>
+            <p_gain>80.0</p_gain>
+            <i_gain>0.0</i_gain>
+            <d_gain>5.0</d_gain>
         </plugin>
         <!-- Expansion Joints Controller -->
@@ -265,14 +348,6 @@
             <joint_name>expansion_joint_left</joint_name>
             <joint_name>expansion_joint_right</joint_name>
-            <p_gain>50000.0</p_gain>
-            <i_gain>1000.0</i_gain>
-            <d_gain>500.0</d_gain>
-        </plugin>
-        <!-- Arm Joints Controller -->
-        <plugin filename="libignition-gazebo-joint-controller-system.so" name="ignition::gazebo::systems::JointController">
-            <joint_name>joint_pitch</joint_name>
-            <joint_name>joint_yaw</joint_name>
-            <p_gain>500.0</p_gain>
-            <i_gain>50.0</i_gain>
+            <p_gain>150.0</p_gain>
+            <i_gain>0.0</i_gain>
             <d_gain>10.0</d_gain>
         </plugin>

Commit message: add Explain.md to describe the project and its components

File: src/simple_car_sim/urdf/robot.urdf.xacro (robot description, xacro)
@@ -4,18 +4,19 @@
     <!--                     1. 属性与常数定义                      -->
     <!-- ========================================================== -->
-    <!-- 尺寸参数 (单位: 米) - 放大 3 倍 -->
-    <xacro:property name="body_len" value="0.75" />
-    <xacro:property name="body_width" value="0.54" />
-    <xacro:property name="body_height" value="0.54" />
-    <xacro:property name="wheel_radius" value="0.18" />
-    <xacro:property name="wheel_width" value="0.15" />
-    <xacro:property name="wheel_offset" value="0.36" /> <!-- 轮子离中心的距离 -->
-    <xacro:property name="leg_radius" value="0.045" />
-    <xacro:property name="leg_length" value="0.3" />
-    <!-- 质量参数 (用于惯性矩阵计算) - 增加质量 -->
-    <xacro:property name="mass_body" value="20.0" />
-    <xacro:property name="mass_wheel" value="2.0" />
-    <xacro:property name="mass_leg" value="1.0" />
-    <!-- 材质颜色 -->
+    <!-- 定义机器人各部分的尺寸、质量等参数，方便统一修改 -->
+    <!-- 尺寸参数 (单位: 米) - 放大 3 倍以适应管道环境 -->
+    <xacro:property name="body_len" value="0.75" />  <!-- 车身长度: 机器人的主体框架长度 -->
+    <xacro:property name="body_width" value="0.54" /> <!-- 车身宽度: 机器人的主体框架宽度 -->
+    <xacro:property name="body_height" value="0.54" /> <!-- 车身高度: 机器人的主体框架高度 -->
+    <xacro:property name="wheel_radius" value="0.18" /> <!-- 轮子半径: 驱动轮的大小 -->
+    <xacro:property name="wheel_width" value="0.15" /> <!-- 轮子宽度: 驱动轮的接触面宽度 -->
+    <xacro:property name="wheel_offset" value="0.36" /> <!-- 轮子离中心的偏移距离 (半宽 + 间隙) -->
+    <xacro:property name="leg_radius" value="0.045" /> <!-- 支撑腿半径: 伸缩腿的粗细 -->
+    <xacro:property name="leg_length" value="0.3" />   <!-- 支撑腿长度: 伸缩腿的初始长度 -->
+    <!-- 质量参数 (用于惯性矩阵计算) - 增加质量以增加物理仿真的稳定性 -->
+    <xacro:property name="mass_body" value="20.0" />  <!-- 车身质量 -->
+    <xacro:property name="mass_wheel" value="2.0" />  <!-- 轮子质量 -->
+    <xacro:property name="mass_leg" value="1.0" />    <!-- 腿部质量 -->
+    <!-- 材质颜色定义 (用于 RViz 可视化) -->
     <material name="blue">
         <color rgba="0.0 0.4 0.8 1.0"/>
@@ -33,5 +34,7 @@
     <!--                     2. 通用宏定义 (Macros)                 -->
     <!-- ========================================================== -->
+    <!-- 使用宏来简化重复代码，特别是对于对称结构 -->
     <!-- 惯性矩阵宏: 盒子 -->
+    <!-- 根据质量和尺寸计算盒子的转动惯量矩阵，用于Gazebo物理引擎计算 -->
     <xacro:macro name="box_inertial" params="mass x y z">
         <inertial>
@@ -43,4 +46,5 @@
     </xacro:macro>
     <!-- 惯性矩阵宏: 圆柱 -->
+    <!-- 根据质量、半径和高度计算圆柱体的转动惯量矩阵 (假设圆柱轴沿Z轴) -->
     <xacro:macro name="cylinder_inertial" params="mass r h">
         <inertial>
@@ -55,4 +59,5 @@
     <!-- ========================================================== -->
     <!-- Base Link: 机器人的主体 (驱动节盒子) -->
+    <!-- 它是整个机器人的根坐标系 -->
     <link name="base_link">
         <visual>
@@ -72,7 +77,8 @@
     </link>
     <!-- 驱动轮宏定义 (带伸缩) -->
-    <!-- 参数: location(位置名称), xyz_offset(初始位置), rpy_offset(旋转), axis_dir(伸缩方向) -->
+    <!-- 创建一个带有伸缩机构和两个驱动轮（前后）的组件 -->
+    <!-- 参数: location(位置名称: top/bottom/left/right), xyz_offset(初始位置), rpy_offset(旋转), axis_dir(伸缩方向) -->
     <xacro:macro name="expandable_drive_wheel" params="location xyz_offset rpy_offset">
-        <!-- 伸缩腿连杆 -->
+        <!-- 伸缩腿连杆: 连接主体和轮架的中间件 -->
         <link name="drive_leg_${location}_link">
             <visual>
@@ -83,5 +89,5 @@
             <xacro:box_inertial mass="0.2" x="0.05" y="0.05" z="0.1"/>
         </link>
-        <!-- 伸缩关节 -->
+        <!-- 伸缩关节: 棱柱关节 (prismatic)，允许沿Z轴直线移动 -->
         <joint name="drive_expansion_joint_${location}" type="prismatic">
             <parent link="base_link"/>
@@ -90,7 +96,7 @@
             <axis xyz="0 0 1"/> <!-- 沿局部Z轴伸缩 -->
             <limit lower="0.0" upper="0.8" effort="5000.0" velocity="0.5"/>
-            <dynamics damping="5.0" friction="0.5"/>
-        </joint>
-        <!-- Bogie Link (连接两个轮子的支架) -->
+            <dynamics damping="5.0" friction="0.5"/> <!-- 增加阻尼和摩擦以模拟真实物理特性 -->
+        </joint>
+        <!-- Bogie Link (转向架/轮架): 连接两个轮子的支架 -->
         <link name="drive_bogie_${location}_link">
             <visual>
@@ -100,4 +106,5 @@
             <xacro:box_inertial mass="0.5" x="0.6" y="0.05" z="0.05"/>
         </link>
+        <!-- 固定关节连接腿和轮架 -->
         <joint name="drive_bogie_joint_${location}" type="fixed">
             <parent link="drive_leg_${location}_link"/>
@@ -105,17 +112,18 @@
             <origin xyz="0 0 0.1" rpy="0 0 0"/>
         </joint>
-        <!-- Front Wheel -->
+        <!-- Front Wheel (前轮) -->
         <link name="drive_wheel_${location}_front_link">
             <visual>
                 <geometry><cylinder radius="${wheel_radius}" length="${wheel_width}"/></geometry>
+                <origin rpy="${pi/2} 0 0"/> <!-- 旋转圆柱体使其平躺为车轮状 -->
+                <material name="black"/>
+            </visual>
+            <collision>
+                <geometry><sphere radius="${wheel_radius}"/></geometry> <!-- 使用球体碰撞优化物理计算稳定性 -->
                 <origin rpy="${pi/2} 0 0"/>
-                <material name="black"/>
-            </visual>
-            <collision>
-                <geometry><sphere radius="${wheel_radius}"/></geometry>
-                <origin rpy="${pi/2} 0 0"/>
             </collision>
             <xacro:cylinder_inertial mass="${mass_wheel}" r="${wheel_radius}" h="${wheel_width}"/>
         </link>
+        <!-- Gazebo 物理属性: 高摩擦力，防止打滑 -->
         <gazebo reference="drive_wheel_${location}_front_link">
             <mu1>4.0</mu1>
@@ -125,13 +133,14 @@
             <minDepth>0.001</minDepth>
         </gazebo>
+        <!-- 轮子驱动关节: 连续旋转关节 -->
         <joint name="drive_wheel_${location}_front_joint" type="continuous">
             <parent link="drive_bogie_${location}_link"/>
             <child link="drive_wheel_${location}_front_link"/>
             <origin xyz="0.25 0 0" rpy="0 0 0"/>
-            <axis xyz="0 1 0"/>
+            <axis xyz="0 1 0"/> <!-- 绕Y轴旋转 -->
             <limit effort="1000.0" velocity="20.0"/>
             <dynamics damping="0.5" friction="0.2"/>
         </joint>
-        <!-- Rear Wheel -->
+        <!-- Rear Wheel (后轮) - 结构同前轮 -->
         <link name="drive_wheel_${location}_rear_link">
             <visual>
@@ -162,16 +171,17 @@
         </joint>
     </xacro:macro>
-    <!-- 实例化4个可伸缩驱动轮 -->
-    <!-- Top Wheel -->
+    <!-- 实例化4个可伸缩驱动轮组件 -->
+    <!-- Top Wheel (顶部轮组) -->
     <xacro:expandable_drive_wheel location="top" xyz_offset="0 0 ${wheel_offset}" rpy_offset="0 0 0"/>
-    <!-- Bottom Wheel -->
+    <!-- Bottom Wheel (底部轮组, 翻转180度) -->
     <xacro:expandable_drive_wheel location="bottom" xyz_offset="0 0 -${wheel_offset}" rpy_offset="${pi} 0 0"/>
-    <!-- Left Wheel -->
+    <!-- Left Wheel (左侧轮组, 翻转-90度) -->
     <xacro:expandable_drive_wheel location="left" xyz_offset="0 ${wheel_offset} 0" rpy_offset="-${pi/2} 0 0"/>
-    <!-- Right Wheel -->
+    <!-- Right Wheel (右侧轮组, 翻转90度) -->
     <xacro:expandable_drive_wheel location="right" xyz_offset="0 -${wheel_offset} 0" rpy_offset="${pi/2} 0 0"/>
     <!-- ========================================================== -->
     <!--             4. 机械臂连接节 (Joint Section - Middle)       -->
     <!-- ========================================================== -->
+    <!-- 连接前后两部分车身的万向节结构 -->
     <!-- 中间虚拟连接杆 (Universal Joint Center) -->
     <link name="universal_joint_link">
@@ -220,4 +230,5 @@
     <!--            5. 功能节 (Functional Section - Left)           -->
     <!-- ========================================================== -->
+    <!-- 后半部分，配有被动轮和伸缩机构，用于支撑和随动 -->
     <!-- 伸缩腿宏定义 (Prismatic Leg + Passive Wheel) -->
     <!-- 参数: suffix(名称后缀), xyz_offset(位置), rpy_offset(旋转) -->
@@ -264,5 +275,5 @@
             <origin xyz="0 0 ${leg_length}" rpy="0 0 0"/>
         </joint>
-        <!-- Front Passive Wheel -->
+        <!-- Front Passive Wheel (前被动轮) - 使用球形万向轮简化 -->
         <link name="passive_wheel_${suffix}_front_link">
             <visual>
@@ -275,4 +286,5 @@
             <xacro:box_inertial mass="0.1" x="0.08" y="0.08" z="0.08"/>
         </link>
+        <!-- 被动轮几乎无摩擦，为了让它顺滑移动 -->
         <gazebo reference="passive_wheel_${suffix}_front_link">
             <mu1>0.001</mu1>
@@ -287,5 +299,5 @@
             <axis xyz="0 1 0"/>
         </joint>
-        <!-- Rear Passive Wheel -->
+        <!-- Rear Passive Wheel (后被动轮) -->
         <link name="passive_wheel_${suffix}_rear_link">
             <visual>
@@ -324,5 +336,6 @@
     <!-- ========================================================== -->
     <gazebo>
-        <!-- Drive Wheels Controller -->
+        <!-- Drive Wheels Controller (驱动轮控制器) -->
+        <!-- 用于发布 cmd_vel 来控制关节速度 -->
         <plugin filename="libignition-gazebo-joint-controller-system.so" name="ignition::gazebo::systems::JointController">
             <joint_name>drive_wheel_top_front_joint</joint_name>
@@ -338,5 +351,7 @@
             <d_gain>5.0</d_gain>
         </plugin>
-        <!-- Expansion Joints Controller -->
+        <!-- Expansion Joints Controller (伸缩关节控制器) -->
+        <!-- 用于控制伸缩腿的长度 (力/位置伺服) -->
+        <!-- 注意：这里配置了 P 增益，说明是位置控制或者有位置反馈 -->
         <plugin filename="libignition-gazebo-joint-controller-system.so" name="ignition::gazebo::systems::JointController">
             <joint_name>drive_expansion_joint_top</joint_name>
