Commit message: 20260128

File: src/simple_car_sim/urdf/robot.urdf.xacro (robot description, xacro)
@@ -5,5 +5,5 @@
     <!-- ========================================================== -->
     <!-- 定义机器人各部分的尺寸、质量等参数，方便统一修改 -->
-    <!-- 尺寸参数 (单位: 米) - 放大 3 倍以适应管道环境 -->
+    <!-- 尺寸参数 (单位: 米) -->
     <xacro:property name="body_len" value="0.75" />  <!-- 车身长度: 机器人的主体框架长度 -->
     <xacro:property name="body_width" value="0.54" /> <!-- 车身宽度: 机器人的主体框架宽度 -->
@@ -11,7 +11,8 @@
     <xacro:property name="wheel_radius" value="0.18" /> <!-- 轮子半径: 驱动轮的大小 -->
     <xacro:property name="wheel_width" value="0.15" /> <!-- 轮子宽度: 驱动轮的接触面宽度 -->
-    <xacro:property name="wheel_offset" value="0.36" /> <!-- 轮子离中心的偏移距离 (半宽 + 间隙) -->
+    <xacro:property name="wheel_offset" value="0.35" /> <!-- 轮子离中心的偏移距离 (半宽 + 间隙) -->
+    <xacro:property name="wheel_interval" value="0.25" /> <!-- 轮子距离中心轴线距离 -->
     <xacro:property name="leg_radius" value="0.045" /> <!-- 支撑腿半径: 伸缩腿的粗细 -->
-    <xacro:property name="leg_length" value="0.3" />   <!-- 支撑腿长度: 伸缩腿的初始长度 -->
+    <xacro:property name="leg_length" value="0.45" />   <!-- 支撑腿长度: 伸缩腿的初始长度 -->
     <!-- 质量参数 (用于惯性矩阵计算) - 增加质量以增加物理仿真的稳定性 -->
     <xacro:property name="mass_body" value="20.0" />  <!-- 车身质量 -->
@@ -62,5 +63,5 @@
     <link name="base_link">
         <visual>
-            <origin xyz="0 0 0" rpy="0 0 0"/>
+            <origin xyz="0 0 0" rpy="${pi/4} 0 0"/>
             <geometry>
                 <box size="${body_len} ${body_width} ${body_height}"/>
@@ -69,5 +70,5 @@
         </visual>
         <collision>
-            <origin xyz="0 0 0" rpy="0 0 0"/>
+            <origin xyz="0 0 0" rpy="${pi/4} 0 0"/>
             <geometry>
                 <box size="${body_len} ${body_width} ${body_height}"/>
@@ -98,4 +99,12 @@
             <dynamics damping="5.0" friction="0.5"/> <!-- 增加阻尼和摩擦以模拟真实物理特性 -->
         </joint>
+        <!-- Drive Expansion Plugin (Drive Section) - Velocity Control (Restored) -->
+        <gazebo>
+            <plugin filename="libignition-gazebo-joint-controller-system.so" name="ignition::gazebo::systems::JointController">
+                <joint_name>drive_expansion_joint_${location}</joint_name>
+                <i_max>1000</i_max>
+                <i_min>-1000</i_min>
+            </plugin>
+        </gazebo>
         <!-- Bogie Link (转向架/轮架): 连接两个轮子的支架 -->
         <link name="drive_bogie_${location}_link">
@@ -137,5 +146,5 @@
             <parent link="drive_bogie_${location}_link"/>
             <child link="drive_wheel_${location}_front_link"/>
-            <origin xyz="0.25 0 0" rpy="0 0 0"/>
+            <origin xyz="${wheel_interval} 0 0" rpy="0 0 0"/>
             <axis xyz="0 1 0"/> <!-- 绕Y轴旋转 -->
             <limit effort="1000.0" velocity="20.0"/>
@@ -165,5 +174,5 @@
             <parent link="drive_bogie_${location}_link"/>
             <child link="drive_wheel_${location}_rear_link"/>
-            <origin xyz="-0.25 0 0" rpy="0 0 0"/>
+            <origin xyz="-${wheel_interval} 0 0" rpy="0 0 0"/>
             <axis xyz="0 1 0"/>
             <limit effort="1000.0" velocity="20.0"/>
@@ -196,6 +205,6 @@
         <parent link="base_link"/>
         <child link="universal_joint_link"/>
-        <origin xyz="-${body_len/2 + 0.08} 0 0" rpy="0 0 0"/>
-        <axis xyz="0 1 0"/>
+        <origin xyz="-${body_len/2 + 0.12} 0 0" rpy="0 0 0"/>
+        <axis xyz="0 0 1"/>
         <limit lower="-1.57" upper="1.57" effort="100.0" velocity="0.5"/>
         <dynamics damping="3.0" friction="0.2"/>
@@ -222,6 +231,6 @@
         <parent link="universal_joint_link"/>
         <child link="func_base_link"/>
-        <origin xyz="-0.12 0 0" rpy="0 0 0"/>
-        <axis xyz="0 0 1"/>
+        <origin xyz="-0.12 0 0" rpy="${pi/4} 0 0"/>
+        <axis xyz="0 ${pi/4} ${pi/4}"/>
         <limit lower="-1.57" upper="1.57" effort="100.0" velocity="0.5"/>
         <dynamics damping="3.0" friction="0.2"/>
@@ -262,11 +271,8 @@
             <dynamics damping="5.0" friction="0.5"/>
         </joint>
-        <!-- Expansion Joint Plugin (Functional Section) -->
+        <!-- Expansion Joint Plugin (Functional Section) - Velocity Control (Restored) -->
          <gazebo>
             <plugin filename="libignition-gazebo-joint-controller-system.so" name="ignition::gazebo::systems::JointController">
                 <joint_name>expansion_joint_${suffix}</joint_name>
-                <p_gain>5000.0</p_gain>
-                <i_gain>100.0</i_gain>
-                <d_gain>50.0</d_gain>
                 <i_max>1000</i_max>
                 <i_min>-1000</i_min>
@@ -336,11 +342,11 @@
     <!-- 实例化4个伸缩腿 -->
     <!-- Top Leg (朝上 +Z) -->
-    <xacro:expansion_leg suffix="top" xyz_offset="-0.25 0 ${body_height/2}" rpy_offset="0 0 0" axis_dir="0 0 1"/>
+    <xacro:expansion_leg suffix="top" xyz_offset="-${body_len/2} 0 ${body_height/2}" rpy_offset="0 0 0" axis_dir="0 0 1"/>
     <!-- Bottom Leg (朝下 -Z) -> 旋转180度使Z轴朝下 -->
-    <xacro:expansion_leg suffix="bottom" xyz_offset="-0.25 0 -${body_height/2}" rpy_offset="${pi} 0 0" axis_dir="0 0 1"/>
+    <xacro:expansion_leg suffix="bottom" xyz_offset="-${body_len/2} 0 -${body_height/2}" rpy_offset="${pi} 0 0" axis_dir="0 0 1"/>
     <!-- Left Leg (朝左 +Y) -> 绕X轴转-90度使Z轴朝左 -->
-    <xacro:expansion_leg suffix="left" xyz_offset="-0.25 ${body_width/2} 0" rpy_offset="-${pi/2} 0 0" axis_dir="0 0 1"/>
+    <xacro:expansion_leg suffix="left" xyz_offset="-${body_len/2} ${body_width/2} 0" rpy_offset="-${pi/2} 0 0" axis_dir="0 0 1"/>
     <!-- Right Leg (朝右 -Y) -> 绕X轴转+90度使Z轴朝右 -->
-    <xacro:expansion_leg suffix="right" xyz_offset="-0.25 -${body_width/2} 0" rpy_offset="${pi/2} 0 0" axis_dir="0 0 1"/>
+    <xacro:expansion_leg suffix="right" xyz_offset="-${body_len/2} -${body_width/2} 0" rpy_offset="${pi/2} 0 0" axis_dir="0 0 1"/>
     <!-- ========================================================== -->
     <!--                     6. Gazebo Plugins                      -->
@@ -359,21 +365,5 @@
             <initial_velocity>0.0</initial_velocity>
         </plugin>
-        <!-- Expansion Joints Controller (伸缩关节控制器) -->
-        <plugin filename="libignition-gazebo-joint-controller-system.so" name="ignition::gazebo::systems::JointController">
-            <joint_name>drive_expansion_joint_top</joint_name>
-            <joint_name>drive_expansion_joint_bottom</joint_name>
-            <joint_name>drive_expansion_joint_left</joint_name>
-            <joint_name>drive_expansion_joint_right</joint_name>
-            <joint_name>expansion_joint_top</joint_name>
-            <joint_name>expansion_joint_bottom</joint_name>
-            <joint_name>expansion_joint_left</joint_name>
-            <joint_name>expansion_joint_right</joint_name>
-             <!-- 增加PID增益以确保能撑起机身 (原值 150 太小) -->
-            <p_gain>200.0</p_gain>
-            <i_gain>4.0</i_gain>
-            <d_gain>2.0</d_gain>
-            <i_max>1000</i_max>
-            <i_min>-1000</i_min>
-        </plugin>
+        <!-- Expansion Joints Controller Removed (Moved to macros) -->
         <!-- Odometry Publisher (里程计发布) -->
         <plugin filename="libignition-gazebo-odometry-publisher-system.so" name="ignition::gazebo::systems::OdometryPublisher">
