Commit message: 1234

File: src/simple_car_sim/urdf/robot.urdf.xacro (robot description, xacro)
@@ -1,41 +1,15 @@
 <?xml version="1.0"?>
-<robot name="pipeline_robot" xmlns:xacro="http://www.ros.org/wiki/xacro">
-    <!-- ========================================================== -->
-    <!--                     1. 属性与常数定义                      -->
-    <!-- ========================================================== -->
-    <!-- 定义机器人各部分的尺寸、质量等参数，方便统一修改 -->
-    <!-- 尺寸参数 (单位: 米) -->
-    <xacro:property name="body_len" value="0.75" />  <!-- 车身长度: 机器人的主体框架长度 -->
-    <xacro:property name="body_width" value="0.54" /> <!-- 车身宽度: 机器人的主体框架宽度 -->
-    <xacro:property name="body_height" value="0.54" /> <!-- 车身高度: 机器人的主体框架高度 -->
-    <xacro:property name="wheel_radius" value="0.18" /> <!-- 轮子半径: 驱动轮的大小 -->
-    <xacro:property name="wheel_width" value="0.15" /> <!-- 轮子宽度: 驱动轮的接触面宽度 -->
-    <xacro:property name="wheel_offset" value="0.35" /> <!-- 轮子离中心的偏移距离 (半宽 + 间隙) -->
-    <xacro:property name="wheel_interval" value="0.25" /> <!-- 轮子距离中心轴线距离 -->
-    <xacro:property name="leg_radius" value="0.045" /> <!-- 支撑腿半径: 伸缩腿的粗细 -->
-    <xacro:property name="leg_length" value="0.45" />   <!-- 支撑腿长度: 伸缩腿的初始长度 -->
-    <!-- 质量参数 (用于惯性矩阵计算) - 增加质量以增加物理仿真的稳定性 -->
-    <xacro:property name="mass_body" value="20.0" />  <!-- 车身质量 -->
-    <xacro:property name="mass_wheel" value="2.0" />  <!-- 轮子质量 -->
-    <xacro:property name="mass_leg" value="1.0" />    <!-- 腿部质量 -->
-    <!-- 材质颜色定义 (用于 RViz 可视化) -->
-    <material name="blue">
-        <color rgba="0.0 0.4 0.8 1.0"/>
-    </material>
-    <material name="black">
-        <color rgba="0.1 0.1 0.1 1.0"/>
-    </material>
-    <material name="grey">
-        <color rgba="0.6 0.6 0.6 1.0"/>
-    </material>
-    <material name="orange">
-        <color rgba="1.0 0.5 0.0 1.0"/>
-    </material>
-    <!-- ========================================================== -->
-    <!--                     2. 通用宏定义 (Macros)                 -->
-    <!-- ========================================================== -->
-    <!-- 使用宏来简化重复代码，特别是对于对称结构 -->
-    <!-- 惯性矩阵宏: 盒子 -->
-    <!-- 根据质量和尺寸计算盒子的转动惯量矩阵，用于Gazebo物理引擎计算 -->
+<robot name="simple_car" xmlns:xacro="http://www.ros.org/wiki/xacro">
+    <xacro:property name="body_len" value="0.8" />
+    <xacro:property name="body_width" value="0.6" />
+    <xacro:property name="body_height" value="0.2" />
+    <xacro:property name="wheel_radius" value="0.16" />
+    <xacro:property name="wheel_width" value="0.04" />
+    <xacro:property name="caster_radius" value="0.16" />
+    <xacro:property name="suspension_travel" value="0.10" />
+    <xacro:property name="mass_body" value="10.0" />
+    <xacro:property name="mass_wheel" value="1.0" />
+    <xacro:property name="mass_caster" value="1.0" />
+    <xacro:property name="mass_suspension" value="0.4" />
     <xacro:macro name="box_inertial" params="mass x y z">
         <inertial>
@@ -46,6 +20,4 @@
         </inertial>
     </xacro:macro>
-    <!-- 惯性矩阵宏: 圆柱 -->
-    <!-- 根据质量、半径和高度计算圆柱体的转动惯量矩阵 (假设圆柱轴沿Z轴) -->
     <xacro:macro name="cylinder_inertial" params="mass r h">
         <inertial>
@@ -56,324 +28,152 @@
         </inertial>
     </xacro:macro>
-    <!-- ========================================================== -->
-    <!--               3. 驱动节 (Drive Section - Right)            -->
-    <!-- ========================================================== -->
-    <!-- Base Link: 机器人的主体 (驱动节盒子) -->
-    <!-- 它是整个机器人的根坐标系 -->
+    <xacro:macro name="sphere_inertial" params="mass r">
+        <inertial>
+            <mass value="${mass}" />
+            <inertia ixx="${(2/5) * mass * r*r}" ixy="0.0" ixz="0.0"
+                     iyy="${(2/5) * mass * r*r}" iyz="0.0"
+                     izz="${(2/5) * mass * r*r}" />
+        </inertial>
+    </xacro:macro>
+    <material name="blue"><color rgba="0.0 0.4 0.8 1.0"/></material>
+    <material name="black"><color rgba="0.1 0.1 0.1 1.0"/></material>
+    <material name="grey"><color rgba="0.6 0.6 0.6 1.0"/></material>
+    <link name="dummy_root"/>
+    <joint name="dummy_joint" type="fixed">
+        <parent link="dummy_root"/>
+        <child link="base_link"/>
+    </joint>
+    <!-- Base Link -->
     <link name="base_link">
         <visual>
-            <origin xyz="0 0 0" rpy="${pi/4} 0 0"/>
-            <geometry>
-                <box size="${body_len} ${body_width} ${body_height}"/>
-            </geometry>
+            <origin xyz="0 0 0" rpy="0 0 0"/>
+            <geometry><box size="${body_len} ${body_width} ${body_height}"/></geometry>
             <material name="blue"/>
         </visual>
         <collision>
-            <origin xyz="0 0 0" rpy="${pi/4} 0 0"/>
-            <geometry>
-                <box size="${body_len} ${body_width} ${body_height}"/>
-            </geometry>
+            <origin xyz="0 0 0" rpy="0 0 0"/>
+            <geometry><box size="${body_len} ${body_width} ${body_height}"/></geometry>
         </collision>
         <xacro:box_inertial mass="${mass_body}" x="${body_len}" y="${body_width}" z="${body_height}" />
     </link>
-    <!-- 驱动轮宏定义 (带伸缩) -->
-    <!-- 创建一个带有伸缩机构和两个驱动轮（前后）的组件 -->
-    <!-- 参数: location(位置名称: top/bottom/left/right), xyz_offset(初始位置), rpy_offset(旋转), axis_dir(伸缩方向) -->
-    <xacro:macro name="expandable_drive_wheel" params="location xyz_offset rpy_offset">
-        <!-- 伸缩腿连杆: 连接主体和轮架的中间件 -->
-        <link name="drive_leg_${location}_link">
+    <!-- IMU Sensor Link -->
+    <link name="imu_link"/>
+    <joint name="imu_joint" type="fixed">
+        <parent link="base_link"/>
+        <child link="imu_link"/>
+        <origin xyz="0 0 0" rpy="0 0 0"/>
+    </joint>
+    <gazebo reference="imu_link">
+        <sensor name="imu_sensor" type="imu">
+            <always_on>1</always_on>
+            <update_rate>50</update_rate>
+            <visualize>true</visualize>
+            <topic>/imu</topic>
+        </sensor>
+    </gazebo>
+    <!-- Suspension Macro -->
+    <xacro:macro name="suspension" params="prefix xyz_offset">
+        <link name="suspension_${prefix}_link">
             <visual>
-                <geometry><box size="0.05 0.05 0.1"/></geometry> <!-- 简单的腿部形状 -->
-                <origin xyz="0 0 0.05" rpy="0 0 0"/>
+                <geometry><box size="0.04 0.04 0.10"/></geometry>
                 <material name="grey"/>
             </visual>
-            <xacro:box_inertial mass="0.2" x="0.05" y="0.05" z="0.1"/>
+            <xacro:box_inertial mass="${mass_suspension}" x="0.04" y="0.04" z="0.10"/>
         </link>
-        <!-- 伸缩关节: 棱柱关节 (prismatic)，允许沿Z轴直线移动 -->
-        <joint name="drive_expansion_joint_${location}" type="prismatic">
+        <joint name="suspension_${prefix}_joint" type="prismatic">
             <parent link="base_link"/>
-            <child link="drive_leg_${location}_link"/>
-            <origin xyz="${xyz_offset}" rpy="${rpy_offset}"/>
-            <axis xyz="0 0 1"/> <!-- 沿局部Z轴伸缩 -->
-            <limit lower="0.0" upper="0.8" effort="5000.0" velocity="0.5"/>
-            <dynamics damping="5.0" friction="0.5"/> <!-- 增加阻尼和摩擦以模拟真实物理特性 -->
+            <child link="suspension_${prefix}_link"/>
+            <origin xyz="${xyz_offset}" rpy="0 0 0"/>
+            <axis xyz="0 0 1"/>
+            <limit lower="-${suspension_travel}" upper="${suspension_travel}" effort="500.0" velocity="10.0"/>
+            <!-- Add spring and damping -->
+            <dynamics damping="50.0" friction="0.1" spring_stiffness="2000.0" spring_reference="0.0"/>
         </joint>
-        <!-- Drive Expansion Plugin (Drive Section) - Velocity Control (Restored) -->
-        <gazebo>
-            <plugin filename="libignition-gazebo-joint-controller-system.so" name="ignition::gazebo::systems::JointController">
-                <joint_name>drive_expansion_joint_${location}</joint_name>
-                <i_max>1000</i_max>
-                <i_min>-1000</i_min>
-            </plugin>
-        </gazebo>
-        <!-- Bogie Link (转向架/轮架): 连接两个轮子的支架 -->
-        <link name="drive_bogie_${location}_link">
+    </xacro:macro>
+    <!-- Rear Wheels Macro (Driven) -->
+    <xacro:macro name="rear_wheel" params="prefix xyz_offset">
+        <xacro:suspension prefix="${prefix}" xyz_offset="${xyz_offset}"/>
+        <link name="wheel_${prefix}_link">
             <visual>
-                <geometry><box size="0.6 0.05 0.05"/></geometry>
-                <material name="grey"/>
-            </visual>
-            <xacro:box_inertial mass="0.5" x="0.6" y="0.05" z="0.05"/>
-        </link>
-        <!-- 固定关节连接腿和轮架 -->
-        <joint name="drive_bogie_joint_${location}" type="fixed">
-            <parent link="drive_leg_${location}_link"/>
-            <child link="drive_bogie_${location}_link"/>
-            <origin xyz="0 0 0.1" rpy="0 0 0"/>
-        </joint>
-        <!-- Front Wheel (前轮) -->
-        <link name="drive_wheel_${location}_front_link">
-            <visual>
+                <origin rpy="${pi/2} 0 0"/>
                 <geometry><cylinder radius="${wheel_radius}" length="${wheel_width}"/></geometry>
-                <origin rpy="${pi/2} 0 0"/> <!-- 旋转圆柱体使其平躺为车轮状 -->
                 <material name="black"/>
             </visual>
             <collision>
-                <geometry><sphere radius="${wheel_radius}"/></geometry> <!-- 使用球体碰撞优化物理计算稳定性 -->
                 <origin rpy="${pi/2} 0 0"/>
+                <!-- Using cylinder or sphere for stability -->
+                <geometry><sphere radius="${wheel_radius}"/></geometry>
             </collision>
             <xacro:cylinder_inertial mass="${mass_wheel}" r="${wheel_radius}" h="${wheel_width}"/>
         </link>
-        <!-- Gazebo 物理属性: 高摩擦力，防止打滑 -->
-        <gazebo reference="drive_wheel_${location}_front_link">
-            <mu1>4.0</mu1>
-            <mu2>4.0</mu2>
-            <kp>10000.0</kp>
-            <kd>5.0</kd>
-            <minDepth>0.001</minDepth>
+        <joint name="wheel_${prefix}_joint" type="continuous">
+            <parent link="suspension_${prefix}_link"/>
+            <child link="wheel_${prefix}_link"/>
+            <origin xyz="0 0 -0.10" rpy="0 0 0"/>
+            <axis xyz="0 1 0"/>
+            <limit effort="500.0" velocity="50.0"/>
+            <dynamics damping="0.1" friction="0.05"/>
+        </joint>
+        <gazebo reference="wheel_${prefix}_link">
+            <mu1>1.0</mu1>
+            <mu2>1.0</mu2>
         </gazebo>
-        <!-- 轮子驱动关节: 连续旋转关节 -->
-        <joint name="drive_wheel_${location}_front_joint" type="continuous">
-            <parent link="drive_bogie_${location}_link"/>
-            <child link="drive_wheel_${location}_front_link"/>
-            <origin xyz="${wheel_interval} 0 0" rpy="0 0 0"/>
-            <axis xyz="0 1 0"/> <!-- 绕Y轴旋转 -->
-            <limit effort="1000.0" velocity="20.0"/>
-            <dynamics damping="0.5" friction="0.2"/>
-        </joint>
-        <!-- Rear Wheel (后轮) - 结构同前轮 -->
-        <link name="drive_wheel_${location}_rear_link">
+    </xacro:macro>
+    <!-- Front Casters Macro (Passive, slide balls) -->
+    <xacro:macro name="front_caster" params="prefix xyz_offset">
+        <xacro:suspension prefix="${prefix}" xyz_offset="${xyz_offset}"/>
+        <link name="caster_${prefix}_link">
             <visual>
-                <geometry><cylinder radius="${wheel_radius}" length="${wheel_width}"/></geometry>
-                <origin rpy="${pi/2} 0 0"/>
+                <geometry><sphere radius="${caster_radius}"/></geometry>
                 <material name="black"/>
             </visual>
             <collision>
-                <geometry><sphere radius="${wheel_radius}"/></geometry>
-                <origin rpy="${pi/2} 0 0"/>
+                <geometry><sphere radius="${caster_radius}"/></geometry>
             </collision>
-            <xacro:cylinder_inertial mass="${mass_wheel}" r="${wheel_radius}" h="${wheel_width}"/>
+            <xacro:sphere_inertial mass="${mass_caster}" r="${caster_radius}"/>
         </link>
-        <gazebo reference="drive_wheel_${location}_rear_link">
-            <mu1>4.0</mu1>
-            <mu2>4.0</mu2>
-            <kp>10000.0</kp>
-            <kd>5.0</kd>
-            <minDepth>0.001</minDepth>
+        <joint name="caster_${prefix}_joint" type="fixed">
+            <parent link="suspension_${prefix}_link"/>
+            <child link="caster_${prefix}_link"/>
+            <origin xyz="0 0 -0.10" rpy="0 0 0"/>
+        </joint>
+        <!-- Low friction for casters -->
+        <gazebo reference="caster_${prefix}_link">
+            <mu1>0.0</mu1>
+            <mu2>0.0</mu2>
         </gazebo>
-        <joint name="drive_wheel_${location}_rear_joint" type="continuous">
-            <parent link="drive_bogie_${location}_link"/>
-            <child link="drive_wheel_${location}_rear_link"/>
-            <origin xyz="-${wheel_interval} 0 0" rpy="0 0 0"/>
-            <axis xyz="0 1 0"/>
-            <limit effort="1000.0" velocity="20.0"/>
-            <dynamics damping="0.5" friction="0.2"/>
-        </joint>
     </xacro:macro>
-    <!-- 实例化4个可伸缩驱动轮组件 -->
-    <!-- Top Wheel (顶部轮组) -->
-    <xacro:expandable_drive_wheel location="top" xyz_offset="0 ${wheel_offset} ${wheel_offset}" rpy_offset="-${pi/4} 0 0"/>
-    <!-- Bottom Wheel (底部轮组, 翻转180度) -->
-    <xacro:expandable_drive_wheel location="bottom" xyz_offset="0 ${wheel_offset} -${wheel_offset}" rpy_offset="-${3*pi/4} 0 0"/>
-    <!-- Left Wheel (左侧轮组, 翻转-90度) -->
-    <xacro:expandable_drive_wheel location="left" xyz_offset="0 -${wheel_offset} ${wheel_offset}" rpy_offset="${pi/4} 0 0"/>
-    <!-- Right Wheel (右侧轮组, 翻转90度) -->
-    <xacro:expandable_drive_wheel location="right" xyz_offset="0 -${wheel_offset} -${wheel_offset}" rpy_offset="${3*pi/4} 0 0"/>
-    <!-- ========================================================== -->
-    <!--             4. 机械臂连接节 (Joint Section - Middle)       -->
-    <!-- ========================================================== -->
-    <!-- 连接前后两部分车身的万向节结构 -->
-    <!-- 中间虚拟连接杆 (Universal Joint Center) -->
-    <link name="universal_joint_link">
-        <visual>
-            <geometry><sphere radius="0.08"/></geometry>
-            <material name="grey"/>
-        </visual>
-        <xacro:box_inertial mass="0.5" x="0.1" y="0.1" z="0.1"/>
-    </link>
-    <!-- 关节1: Pitch (俯仰 - 绕Y轴) -->
-    <joint name="joint_pitch" type="revolute">
-        <parent link="base_link"/>
-        <child link="universal_joint_link"/>
-        <origin xyz="-${body_len/2 + 0.12} 0 0" rpy="0 0 0"/>
-        <axis xyz="0 0 1"/>
-        <limit lower="-1.57" upper="1.57" effort="100.0" velocity="0.5"/>
-        <dynamics damping="3.0" friction="0.2"/>
-    </joint>
-    <!-- 功能节的主体基座 -->
-    <link name="func_base_link">
-        <visual>
-            <origin xyz="-${body_len/2} 0 0" rpy="0 0 0"/> <!-- Offset geometry to start after joint -->
-            <geometry>
-                <box size="${body_len} ${body_width} ${body_height}"/>
-            </geometry>
-            <material name="blue"/>
-        </visual>
-        <collision>
-            <origin xyz="-${body_len/2} 0 0" rpy="0 0 0"/>
-            <geometry>
-                <box size="${body_len} ${body_width} ${body_height}"/>
-            </geometry>
-        </collision>
-        <xacro:box_inertial mass="${mass_body}" x="${body_len}" y="${body_width}" z="${body_height}" />
-    </link>
-    <!-- 关节2: Yaw (偏航 - 绕Z轴) -->
-    <joint name="joint_yaw" type="revolute">
-        <parent link="universal_joint_link"/>
-        <child link="func_base_link"/>
-        <origin xyz="-0.12 0 0" rpy="${pi/4} 0 0"/>
-        <axis xyz="0 ${pi/4} ${pi/4}"/>
-        <limit lower="-1.57" upper="1.57" effort="100.0" velocity="0.5"/>
-        <dynamics damping="3.0" friction="0.2"/>
-    </joint>
-    <!-- ========================================================== -->
-    <!--            5. 功能节 (Functional Section - Left)           -->
-    <!-- ========================================================== -->
-    <!-- 后半部分，配有被动轮和伸缩机构，用于支撑和随动 -->
-    <!-- 伸缩腿宏定义 (Prismatic Leg + Passive Wheel) -->
-    <!-- 参数: suffix(名称后缀), xyz_offset(位置), rpy_offset(旋转) -->
-    <xacro:macro name="expansion_leg" params="suffix xyz_offset rpy_offset axis_dir">
-        <!-- 腿部连杆 -->
-        <link name="leg_${suffix}_link">
-            <visual>
-                <geometry>
-                    <cylinder radius="${leg_radius}" length="${leg_length}"/>
-                </geometry>
-                <!-- 腿沿着Z轴方向 -->
-                <origin xyz="0 0 ${leg_length/2}" rpy="0 0 0"/>
-                <material name="orange"/>
-            </visual>
-            <collision>
-                 <geometry>
-                    <cylinder radius="${leg_radius}" length="${leg_length}"/>
-                </geometry>
-                <origin xyz="0 0 ${leg_length/2}" rpy="0 0 0"/>
-            </collision>
-            <xacro:cylinder_inertial mass="${mass_leg}" r="${leg_radius}" h="${leg_length}"/>
-        </link>
-        <!-- 伸缩关节 (Prismatic) - 模拟剪叉张开 -->
-        <joint name="expansion_joint_${suffix}" type="prismatic">
-            <parent link="func_base_link"/>
-            <child link="leg_${suffix}_link"/>
-            <origin xyz="${xyz_offset}" rpy="${rpy_offset}"/>
-            <!-- 沿着局部坐标系的Z轴伸缩 -->
-            <axis xyz="0 0 1"/>
-            <limit lower="0.0" upper="0.8" effort="5000.0" velocity="0.5"/>
-            <dynamics damping="5.0" friction="0.5"/>
-        </joint>
-        <!-- Expansion Joint Plugin (Functional Section) - Velocity Control (Restored) -->
-         <gazebo>
-            <plugin filename="libignition-gazebo-joint-controller-system.so" name="ignition::gazebo::systems::JointController">
-                <joint_name>expansion_joint_${suffix}</joint_name>
-                <i_max>1000</i_max>
-                <i_min>-1000</i_min>
-            </plugin>
-         </gazebo>
-        <!-- Bogie Link (连接两个轮子的支架) -->
-        <link name="passive_bogie_${suffix}_link">
-            <visual>
-                <geometry><box size="0.4 0.05 0.05"/></geometry>
-                <material name="grey"/>
-            </visual>
-            <xacro:box_inertial mass="0.5" x="0.4" y="0.05" z="0.05"/>
-        </link>
-        <joint name="passive_bogie_joint_${suffix}" type="fixed">
-            <parent link="leg_${suffix}_link"/>
-            <child link="passive_bogie_${suffix}_link"/>
-            <origin xyz="0 0 ${leg_length}" rpy="0 0 0"/>
-        </joint>
-        <!-- Front Passive Wheel (前被动轮) - 使用球形万向轮简化 -->
-        <link name="passive_wheel_${suffix}_front_link">
-            <visual>
-                <geometry><sphere radius="0.04"/></geometry>
-                <material name="black"/>
-            </visual>
-             <collision>
-                <geometry><sphere radius="0.04"/></geometry>
-            </collision>
-            <xacro:box_inertial mass="0.1" x="0.08" y="0.08" z="0.08"/>
-        </link>
-        <!-- 被动轮几乎无摩擦，为了让它顺滑移动 -->
-        <gazebo reference="passive_wheel_${suffix}_front_link">
-            <mu1>0.001</mu1>
-            <mu2>0.001</mu2>
-            <kp>1000000.0</kp>
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
Commit message: to_final

File: src/simple_car_sim/urdf/robot.urdf.xacro (robot description, xacro)
@@ -149,4 +149,86 @@
     <xacro:rear_wheel prefix="rl" xyz_offset="-0.30 0.34 -0.20"/>
     <xacro:rear_wheel prefix="rr" xyz_offset="-0.30 -0.34 -0.20"/>
+    <!-- Lidar Link and Sensor -->
+    <link name="lidar_link">
+        <visual>
+            <geometry><cylinder radius="0.05" length="0.05"/></geometry>
+            <material name="black"/>
+        </visual>
+        <collision>
+            <geometry><cylinder radius="0.05" length="0.05"/></geometry>
+        </collision>
+        <xacro:cylinder_inertial mass="0.1" r="0.05" h="0.05"/>
+    </link>
+    <joint name="lidar_joint" type="fixed">
+        <parent link="base_link"/>
+        <child link="lidar_link"/>
+        <origin xyz="0.0 0 0.15" rpy="0 0 0"/>
+    </joint>
+    <gazebo reference="lidar_link">
+        <sensor name='lidar_sensor' type='gpu_lidar'>
+            <pose>0 0 0 0 0 0</pose>
+            <topic>/scan</topic>
+            <update_rate>10</update_rate>
+            <ray>
+                <scan>
+                    <horizontal>
+                        <samples>360</samples>
+                        <resolution>1</resolution>
+                        <min_angle>-3.14159</min_angle>
+                        <max_angle>3.14159</max_angle>
+                    </horizontal>
+                    <vertical>
+                        <samples>1</samples>
+                        <resolution>0.01</resolution>
+                        <min_angle>0</min_angle>
+                        <max_angle>0</max_angle>
+                    </vertical>
+                </scan>
+                <range>
+                    <min>0.08</min>
+                    <max>10.0</max>
+                    <resolution>0.01</resolution>
+                </range>
+            </ray>
+            <always_on>1</always_on>
+            <visualize>true</visualize>
+        </sensor>
+    </gazebo>
+    <!-- Camera Link and Sensor -->
+    <link name="camera_link">
+        <visual>
+            <geometry><box size="0.05 0.05 0.05"/></geometry>
+            <material name="black"/>
+        </visual>
+        <collision>
+            <geometry><box size="0.05 0.05 0.05"/></geometry>
+        </collision>
+        <xacro:box_inertial mass="0.1" x="0.05" y="0.05" z="0.05"/>
+    </link>
+    <joint name="camera_joint" type="fixed">
+        <parent link="base_link"/>
+        <child link="camera_link"/>
+        <origin xyz="0.4 0 0.1" rpy="0 0 0"/>
+    </joint>
+    <gazebo reference="camera_link">
+        <sensor name="camera_sensor" type="camera">
+            <topic>/camera/image_raw</topic>
+            <update_rate>30</update_rate>
+            <camera>
+                <horizontal_fov>1.047</horizontal_fov>
+                <image>
+                    <width>640</width>
+                    <height>480</height>
+                    <format>R8G8B8</format>
+                </image>
+                <clip>
+                    <near>0.1</near>
+                    <far>100</far>
+                </clip>
+            </camera>
+            <always_on>1</always_on>
+            <visualize>true</visualize>
+        </sensor>
+    </gazebo>
     <!-- Gazebo Plugins -->
     <gazebo>
